File: kicad/maulwurf.kicad_pcb (KiCad board)
At the start: 2 copper layers, 63.5 x 70 mm, 24 parts

Commit message: Fix issue with bottom copper outline connection
Parts:
- turned G*** to 0.2 degrees

Commit message: Remove unmasked rings around eyes
Parts:
- turned MASK to 0 degrees
